File: OsseyPad Rev 1.0/OsseyPad.kicad_pcb (KiCad board)
At the start: 4 copper layers, 152.4 x 142.9 mm, 96 parts, among them J1 USB_C_Receptacle_USB2.0, SW1 Rotary_Encoder_Switch, SW2 SW_Push, U1 USBLC6-2SC6, U2 ATmega32U4-MU, Y1 16MHz

Commit message: Updated the case and pcb.
Parts:
- FB1: value 50 @ 100 MHz -> 100 @ 100 MHz
- J1: value USB_C_Receptacle_USB2.0 -> USB_C_U262-161N-4BVC11
- moved J1 2.00 mm to (51.5, 25.3)
- moved C1 0.23 mm to (58.4, 55.8)
Routing:
- net VCC: track 44.1 -> 31.7 mm
- net USB_CONN_D+: track 21.6 -> 18.9 mm
- net GND: track 65.2 -> 67.1 mm
- net Net-(J1-PadA5): track 14.2 -> 12.4 mm
- net USB_CONN_D-: track 21.8 -> 20.3 mm
- net Net-(J1-PadB5): track 19.3 -> 18.0 mm
Other:
- outline, holes or cut-outs redrawn
- board text added: "+"
- board text added: "Designed by Osku Väyrynen 11/01/2021 Rev 1.0"
- board text added: "GND"
- board text added: "JLCJLCJLCJLC"
- board text added: "RESET"
