File: OsseyPad Rev 1.0/OsseyPad.sch (KiCad schematic (older format))
At the start: 95 parts, among them J1 USB_C_Receptacle_USB2.0, SW1 Rotary_Encoder_Switch, SW2 SW_Push, U1 USBLC6-2SC6, U2 ATmega32U4-MU, Y1 16MHz

Commit message: Updated the case and pcb.
Parts:
- removed J1: USB_C_Receptacle_USB2.0, josh-connectors:USB_C_U262-161N-4BVC11, symbol Connector:USB_C_Receptacle_USB2.0
- added J1: USB_C_U262-161N-4BVC11, josh-connectors:USB_C_U262-161N-4BVC11, symbol josh-connector:USB_C_U262-161N-4BVC11
- FB1: value 50 @ 100 MHz -> 100 @ 100 MHz
- MX1: footprint MX_Alps_Hybrid:MX-10U -> MX_Only:MXOnly-1U-NoLED
- U1: value USBLC6-2SC6 -> TPUSBLC6-2SC6
Connections:
- net GND: now also C1.2, C2.2, C3.2, C4.2, C5.2, J1.A1 (GND), J1.A12 (GND), J1.B1 (GND), J1.B12 (GND)
- net USB_CONN_D+: now also J1.A6 (D+), J1.B6 (D+)
- net USB_CONN_D-: now also J1.A7 (D-), J1.B7 (D-)
- net VCC: now also J1.A4 (VBUS), J1.A9 (VBUS), J1.B4 (VBUS), J1.B9 (VBUS)
- net at R10.2: now also J1.A5 (CC1)
- net at R11.2: now also J1.B5 (CC2)
Other:
- moved on the sheet: F1, FB1, R10, R11, U1
