File: OsseyPad Rev 2.0/OsseyPad.sch (KiCad schematic (older format))
At the start: 83 parts, among them SW1 Rotary_Encoder_Switch

Commit message: Worked on with 2.0
Parts:
- added B1: SPARKFUN_PRO_MICRO, SPARKFUN_PRO_MICRO, symbol SparkFun-Boards:SPARKFUN_PRO_MICRO
- C1, C2: value 100n -> 0.1 uf; footprint Capacitor_SMD:C_0603_1608Metric -> Capacitor_THT:C_Axial_L5.1mm_D3.1mm_P7.50mm_Horizontal
- R1, R2, R3, R4: footprint Resistor_SMD:R_0603_1608Metric -> Resistor_THT:R_Axial_DIN0207_L6.3mm_D2.5mm_P7.62mm_Horizontal
Connections:
- net GND: now also B1.23 (GND), B1.3 (GND), B1.4 (GND)
- net ROW3ENTER: now also D24.2 (A), MX23.2 (ROW); no longer D22.2 (A), MX21.2 (ROW)
- net ROW4+: now reaches D16.2 (A), MX15.2 (ROW)
- net ROW4+: now also MX35.2 (ROW)
- net +5V renamed +3V3
- net +3V3: now also B1.21 (VCC)
- net COL3+ renamed COL1+
- net ROW3+: no longer names the net of D10.2 (A), MX9.2 (ROW)
- net ROW3+: no longer MX35.2 (ROW)
- new net: D22.2 (A), MX21.2 (ROW)
Changed lines of the file:
@@
-	1    0    0    -1
-$EndComp
-$Comp
-L power:+5V #PWR01
-U 1 1 60482C76
-P 3350 1200
-F 0 "#PWR01" H 3350 1050 50  0001 C CNN
-F 1 "+5V" H 3365 1373 50  0000 C CNN
-F 2 "" H 3350 1200 50  0001 C CNN
-F 3 "" H 3350 1200 50  0001 C CNN
-	1    3350 1200
-	1    0    0    -1
-$EndComp
-$Comp
-L power:+5V #PWR02
-U 1 1 60473220
-P 3600 1200
-F 0 "#PWR02" H 3600 1050 50  0001 C CNN
-F 1 "+5V" H 3615 1373 50  0000 C CNN
-F 2 "" H 3600 1200 50  0001 C CNN
-F 3 "" H 3600 1200 50  0001 C CNN
-	1    3600 1200
 	1    0    0    -1
 $EndComp
@@
 P 2450 1900
 F 0 "C1" H 2542 1946 50  0000 L CNN
-F 1 "100n" H 2542 1855 50  0000 L CNN
-F 2 "Capacitor_SMD:C_0603_1608Metric" H 2450 1900 50  0001 C CNN
+F 1 "0.1 uf" H 2542 1855 50  0000 L CNN
+F 2 "Capacitor_THT:C_Axial_L5.1mm_D3.1mm_P7.50mm_Horizontal" H 2450 1900 50  0001 C CNN
 F 3 "~" H 2450 1900 50  0001 C CNN
 	1    2450 1900
@@
 P 2850 1900
 F 0 "C2" H 2942 1946 50  0000 L CNN
-F 1 "100n" H 2942 1855 50  0000 L CNN
-F 2 "Capacitor_SMD:C_0603_1608Metric" H 2850 1900 50  0001 C CNN
+F 1 "0.1 uf" H 2942 1855 50  0000 L CNN
+F 2 "Capacitor_THT:C_Axial_L5.1mm_D3.1mm_P7.50mm_Horizontal" H 2850 1900 50  0001 C CNN
 F 3 "~" H 2850 1900 50  0001 C CNN
 	1    2850 1900
@@
 F 0 "R4" V 3100 1700 50  0000 C CNN
 F 1 "10K" V 3000 1700 50  0000 C CNN
-F 2 "Resistor_SMD:R_0603_1608Metric" H 3100 1700 50  0001 C CNN
+F 2 "Resistor_THT:R_Axial_DIN0207_L6.3mm_D2.5mm_P7.62mm_Horizontal" H 3100 1700 50  0001 C CNN
 F 3 "~" H 3100 1700 50  0001 C CNN
 	1    3100 1700
@@
 F 0 "R3" V 3100 1500 50  0000 C CNN
 F 1 "10K" V 2995 1500 50  0000 C CNN
-F 2 "Resistor_SMD:R_0603_1608Metric" H 3100 1500 50  0001 C CNN
+F 2 "Resistor_THT:R_Axial_DIN0207_L6.3mm_D2.5mm_P7.62mm_Horizontal" H 3100 1500 50  0001 C CNN
 F 3 "~" H 3100 1500 50  0001 C CNN
 	1    3100 1500
@@
 F 0 "R2" H 3659 1396 50  0000 L CNN
 F 1 "10K" H 3659 1305 50  0000 L CNN
-F 2 "Resistor_SMD:R_0603_1608Metric" H 3600 1350 50  0001 C CNN
+F 2 "Resistor_THT:R_Axial_DIN0207_L6.3mm_D2.5mm_P7.62mm_Horizontal" H 3600 1350 50  0001 C CNN
 F 3 "~" H 3600 1350 50  0001 C CNN
 	1    3600 1350
@@
 F 0 "R1" H 3409 1396 50  0000 L CNN
 F 1 "10K" H 3409 1305 50  0000 L CNN
-F 2 "Resistor_SMD:R_0603_1608Metric" H 3350 1350 50  0001 C CNN
+F 2 "Resistor_THT:R_Axial_DIN0207_L6.3mm_D2.5mm_P7.62mm_Horizontal" H 3350 1350 50  0001 C CNN
 F 3 "~" H 3350 1350 50  0001 C CNN
 	1    3350 1350
@@
 	4300 3100 4300 3700
 Connection ~ 4300 3100
-Wire Wire Line
-	4050 3100 4250 3100
 Connection ~ 4300 4300
-Wire Wire Line
-	4050 4300 4250 4300
 Wire Wire Line
 	4050 5500 4300 5500
@@
 $EndComp
 Wire Wire Line
-	4050 3700 4300 3700
+	4050 3700 4250 3700
 $Comp
 L MX_Alps_Hybrid:MX-NoLED MX15
@@
 $EndComp
 Text GLabel 4050 6550 2    50   Input ~ 0
-ROW3+
+ROW4+
 $Comp
 L MX_Alps_Hybrid:MX-NoLED MX37
@@
 	3850 7050 4050 7050
 Text GLabel 4050 6350 2    50   Input ~ 0
-COL3+
+COL1+
 Text GLabel 4050 6850 2    50   Input ~ 0
-COL3ENTER
+COL4ENTER
 Text GLabel 2350 7400 2    50   Input ~ 0
 COL10
@@
 	2200 5800 2200 5700
 Connection ~ 2200 5700
-Text GLabel 3800 3400 1    28   Input ~ 0
-ROW3+
-Text GLabel 4150 3050 0    28   Input ~ 0
-COL3+
-Text GLabel 3800 4550 1    28   Input ~ 0
+Text GLabel 3800 3950 1    28   Input ~ 0
+ROW4+
+Text GLabel 4200 3650 0    28   Input ~ 0
+COL1+
+Text GLabel 3800 5200 1    28   Input ~ 0
 ROW3ENTER
-Text GLabel 4250 4250 0    28   Input ~ 0
-COL3ENTER
-Wire Wire Line
-	4250 4250 4250 4300
-Connection ~ 4250 4300
-Wire Wire Line
-	4250 4300 4300 4300
-Wire Wire Line
-	3850 4500 3850 4550
-Wire Wire Line
-	3850 4550 3800 4550
-Connection ~ 3850 4500
-Wire Wire Line
-	4150 3050 4250 3050
-Wire Wire Line
-	4250 3050 4250 3100
-Connection ~ 4250 3100
-Wire Wire Line
-	4250 3100 4300 3100
+Text GLabel 4250 4850 0    28   Input ~ 0
+COL4ENTER
 $Comp
 L Diode:1N4148 D9
@@
 $EndComp
 Wire Wire Line
-	3850 3300 3850 3400
-Wire Wire Line
-	3850 3400 3800 3400
-Connection ~ 3850 3300
-Wire Wire Line
 	3700 5250 4250 5250
 Wire Wire Line
 	4300 4300 4300 4900
 Wire Wire Line
-	4050 4900 4300 4900
+	4050 4900 4250 4900
 Connection ~ 4300 4900
 Wire Wire Line
@@
 Wire Wire Line
 	4250 5250 4800 5250
+Wire Wire Line
+	4050 4300 4300 4300
+Wire Wire Line
+	3800 5200 3850 5200
+Wire Wire Line
+	3850 5200 3850 5100
+Connection ~ 3850 5100
+Wire Wire Line
+	4250 4850 4250 4900
+Connection ~ 4250 4900
+Wire Wire Line
+	4250 4900 4300 4900
+Wire Wire Line
+	4050 3100 4300 3100
+Wire Wire Line
+	3850 3900 3850 4000
+Wire Wire Line
+	3850 4000 3800 4000
+Wire Wire Line
+	3800 4000 3800 3950
+Connection ~ 3850 3900
+Wire Wire Line
+	4200 3650 4250 3650
+Wire Wire Line
+	4250 3650 4250 3700
+Connection ~ 4250 3700
+Wire Wire Line
+	4250 3700 4300 3700
+$Comp
+L power:+3.3V #PWR0101
+U 1 1 602774ED
+P 3350 1200
+F 0 "#PWR0101" H 3350 1050 50  0001 C CNN
+F 1 "+3.3V" H 3365 1373 50  0000 C CNN
+F 2 "" H 3350 1200 50  0001 C CNN
+F 3 "" H 3350 1200 50  0001 C CNN
+	1    3350 1200
+	1    0    0    -1
+$EndComp
+$Comp
+L power:+3.3V #PWR0102
+U 1 1 60277CF8
+P 3600 1200
+F 0 "#PWR0102" H 3600 1050 50  0001 C CNN
+F 1 "+3.3V" H 3615 1373 50  0000 C CNN
+F 2 "" H 3600 1200 50  0001 C CNN
+F 3 "" H 3600 1200 50  0001 C CNN
+	1    3600 1200
+	1    0    0    -1
+$EndComp
+$Comp
+L SparkFun-Boards:SPARKFUN_PRO_MICRO B1
+U 1 1 6016D8A9
+P 9450 3350
+F 0 "B1" H 9450 4260 45  0000 C CNN
+F 1 "SPARKFUN_PRO_MICRO" H 9450 4176 45  0000 C CNN
+F 2 "SPARKFUN_PRO_MICRO" H 9450 4150 20  0001 C CNN
+F 3 "" H 9450 3350 50  0001 C CNN
+F 4 "XXX-00000" H 9450 4081 60  0000 C CNN "Field4"
+	1    9450 3350
+	1    0    0    -1
+$EndComp
+Wire Wire Line
+	9900 2900 10000 2900
+Wire Wire Line
+	10000 2900 10000 2950
+Wire Wire Line
+	9000 3100 8900 3100
+Wire Wire Line
+	8900 3100 8900 3150
+Wire Wire Line
+	9000 3000 8900 3000
+Wire Wire Line
+	8900 3000 8900 3100
+Connection ~ 8900 3100
+$Comp
+L power:GND #PWR?
+U 1 1 601AEF13
+P 8900 3150
+F 0 "#PWR?" H 8900 2900 50  0001 C CNN
+F 1 "GND" H 8905 2977 50  0000 C CNN
+F 2 "" H 8900 3150 50  0001 C CNN
+F 3 "" H 8900 3150 50  0001 C CNN
+	1    8900 3150
+	1    0    0    -1
+$EndComp
+$Comp
+L power:GND #PWR?
+U 1 1 601AF2A1
+P 10000 2950
+F 0 "#PWR?" H 10000 2700 50  0001 C CNN
+F 1 "GND" H 10000 2950 50  0000 C CNN
+F 2 "" H 10000 2950 50  0001 C CNN
+F 3 "" H 10000 2950 50  0001 C CNN
+	1    10000 2950
+	1    0    0    -1
+$EndComp
+Wire Wire Line
+	9900 3100 10150 3100
+Wire Wire Line
+	10150 3100 10150 3050
+$Comp
+L power:+3.3V #PWR?
+U 1 1 601CC952
+P 10150 3050
+F 0 "#PWR?" H 10150 2900 50  0001 C CNN
+F 1 "+3.3V" H 10165 3223 50  0000 C CNN
+F 2 "" H 10150 3050 50  0001 C CNN
+F 3 "" H 10150 3050 50  0001 C CNN
+	1    10150 3050
+	1    0    0    -1
+$EndComp
 $EndSCHEMATC

Commit message: Worked on Rev 2.0.
Connections:
- net COL1+ is gone; now on net COL4: MX15.1 (COL), MX21.1 (COL), MX23.1 (COL), MX33.1 (COL), MX35.1 (COL), MX36.1 (COL), MX4.1 (COL), MX9.1 (COL)
- net COL0: now also B1.13 (*10)
- net COL1: now also B1.11 (8)
- net COL2: now also B1.10 (7)
- net COL3: now also B1.9 (*6)
- net COL5: now also B1.7 (4)
- net ENC_1_A: now also B1.5 (2)
- net ENC_1_B: now also B1.12 (*9)
- net ROW0: now also B1.6 (*3)
- net ROW1: now also B1.16 (13(SCK))
- net ROW2: now also B1.17 (A0)
- net ROW3: now also B1.18 (A1)
- net ROW4: now also B1.19 (A2)
- net ROW5: now also B1.20 (A3)
- net COL4: now reaches B1.8 (*5)
- net +3V3 renamed +5V
- net ROW3ENTER renamed ROW4ENTER
- net ROW4+ renamed ROW2+
- no-connect marks 0 -> 6
Changed lines of the file:
@@
 $EndComp
 Text GLabel 4050 6550 2    50   Input ~ 0
-ROW4+
+ROW2+
 $Comp
 L MX_Alps_Hybrid:MX-NoLED MX37
@@
 $EndComp
 Text GLabel 4050 7050 2    50   Input ~ 0
-ROW3ENTER
+ROW4ENTER
 Wire Wire Line
 	2100 5500 2100 6050
@@
 	3850 7050 4050 7050
 Text GLabel 4050 6350 2    50   Input ~ 0
-COL1+
+COL4+
 Text GLabel 4050 6850 2    50   Input ~ 0
 COL4ENTER
@@
 Connection ~ 2200 5700
 Text GLabel 3800 3950 1    28   Input ~ 0
-ROW4+
+ROW2+
 Text GLabel 4200 3650 0    28   Input ~ 0
-COL1+
+COL4+
 Text GLabel 3800 5200 1    28   Input ~ 0
-ROW3ENTER
+ROW4ENTER
 Text GLabel 4250 4850 0    28   Input ~ 0
 COL4ENTER
@@
 	4250 3700 4300 3700
 $Comp
-L power:+3.3V #PWR0101
-U 1 1 602774ED
-P 3350 1200
-F 0 "#PWR0101" H 3350 1050 50  0001 C CNN
-F 1 "+3.3V" H 3365 1373 50  0000 C CNN
-F 2 "" H 3350 1200 50  0001 C CNN
-F 3 "" H 3350 1200 50  0001 C CNN
-	1    3350 1200
-	1    0    0    -1
-$EndComp
-$Comp
-L power:+3.3V #PWR0102
-U 1 1 60277CF8
-P 3600 1200
-F 0 "#PWR0102" H 3600 1050 50  0001 C CNN
-F 1 "+3.3V" H 3615 1373 50  0000 C CNN
-F 2 "" H 3600 1200 50  0001 C CNN
-F 3 "" H 3600 1200 50  0001 C CNN
-	1    3600 1200
-	1    0    0    -1
-$EndComp
-$Comp
 L SparkFun-Boards:SPARKFUN_PRO_MICRO B1
 U 1 1 6016D8A9
@@
 F 1 "SPARKFUN_PRO_MICRO" H 9450 4176 45  0000 C CNN
 F 2 "SPARKFUN_PRO_MICRO" H 9450 4150 20  0001 C CNN
-F 3 "" H 9450 3350 50  0001 C CNN
+F 3 "https://cdn.sparkfun.com/assets/f/d/8/0/d/ProMicro16MHzv2.pdf" H 9450 3350 50  0001 C CNN
 F 4 "XXX-00000" H 9450 4081 60  0000 C CNN "Field4"
 	1    9450 3350
@@
 	9000 3100 8900 3100
 Wire Wire Line
-	8900 3100 8900 3150
+	8100 3100 8100 3150
 Wire Wire Line
 	9000 3000 8900 3000
 Wire Wire Line
 	8900 3000 8900 3100
-Connection ~ 8900 3100
-$Comp
-L power:GND #PWR?
+$Comp
+L power:GND #PWR07
 U 1 1 601AEF13
-P 8900 3150
-F 0 "#PWR?" H 8900 2900 50  0001 C CNN
-F 1 "GND" H 8905 2977 50  0000 C CNN
-F 2 "" H 8900 3150 50  0001 C CNN
-F 3 "" H 8900 3150 50  0001 C CNN
-	1    8900 3150
-	1    0    0    -1
-$EndComp
-$Comp
-L power:GND #PWR?
+P 8100 3150
+F 0 "#PWR07" H 8100 2900 50  0001 C CNN
+F 1 "GND" H 8105 2977 50  0000 C CNN
+F 2 "" H 8100 3150 50  0001 C CNN
+F 3 "" H 8100 3150 50  0001 C CNN
+	1    8100 3150
+	1    0    0    -1
+$EndComp
+$Comp
+L power:GND #PWR01
 U 1 1 601AF2A1
 P 10000 2950
-F 0 "#PWR?" H 10000 2700 50  0001 C CNN
+F 0 "#PWR01" H 10000 2700 50  0001 C CNN
 F 1 "GND" H 10000 2950 50  0000 C CNN
 F 2 "" H 10000 2950 50  0001 C CNN
@@
 Wire Wire Line
 	10150 3100 10150 3050
-$Comp
-L power:+3.3V #PWR?
-U 1 1 601CC952
+Text GLabel 9900 3200 2    50   Input ~ 0
+ROW5
+Text GLabel 9900 3300 2    50   Input ~ 0
+ROW4
+Text GLabel 9900 3400 2    50   Input ~ 0
+ROW3
+Text GLabel 9900 3500 2    50   Input ~ 0
+ROW2
+Text GLabel 9900 3600 2    50   Input ~ 0
+ROW1
+Text GLabel 9000 3300 0    50   Input ~ 0
+ROW0
+Wire Wire Line
+	8900 3100 8100 3100
+Connection ~ 8900 3100
+$Comp
+L power:+5V #PWR02
+U 1 1 6026AD68
 P 10150 3050
-F 0 "#PWR?" H 10150 2900 50  0001 C CNN
-F 1 "+3.3V" H 10165 3223 50  0000 C CNN
+F 0 "#PWR02" H 10150 2900 50  0001 C CNN
+F 1 "+5V" H 10165 3223 50  0000 C CNN
 F 2 "" H 10150 3050 50  0001 C CNN
 F 3 "" H 10150 3050 50  0001 C CNN
@@
 	1    0    0    -1
 $EndComp
+$Comp
+L power:+5V #PWR09
+U 1 1 6027389E
+P 3600 1200
+F 0 "#PWR09" H 3600 1050 50  0001 C CNN
+F 1 "+5V" H 3615 1373 50  0000 C CNN
+F 2 "" H 3600 1200 50  0001 C CNN
+F 3 "" H 3600 1200 50  0001 C CNN
+	1    3600 1200
+	1    0    0    -1
+$EndComp
+$Comp
+L power:+5V #PWR08
+U 1 1 60281485
+P 3350 1200
+F 0 "#PWR08" H 3350 1050 50  0001 C CNN
+F 1 "+5V" H 3365 1373 50  0000 C CNN
+F 2 "" H 3350 1200 50  0001 C CNN
+F 3 "" H 3350 1200 50  0001 C CNN
+	1    3350 1200
+	1    0    0    -1
+$EndComp
+Text GLabel 9900 3900 2    50   Input ~ 0
+COL0
+Text GLabel 9000 3800 0    50   Input ~ 0
+COL1
+Text GLabel 9000 3700 0    50   Input ~ 0
+COL2
+Text GLabel 9000 3600 0    50   Input ~ 0
+COL3
+Text GLabel 9000 3500 0    50   Input ~ 0
+COL4
+Text GLabel 9000 3400 0    50   Input ~ 0
+COL5
+Text GLabel 9000 3900 0    50   Input ~ 0
+ENC_1_B
+Text GLabel 9000 3200 0    50   Input ~ 0
+ENC_1_A
+NoConn ~ 9900 3700
+NoConn ~ 9900 3800
+NoConn ~ 9900 3000
+NoConn ~ 9900 2800
+NoConn ~ 9000 2800
+NoConn ~ 9000 2900
 $EndSCHEMATC

Commit message: Worked on the pcb design.
Parts:
- B1: footprint SPARKFUN_PRO_MICRO -> OsseyPad:SPARKFUN_PRO_MICRO_OsseyPad
Changed lines of the file:
@@
 F 0 "B1" H 9450 4260 45  0000 C CNN
 F 1 "SPARKFUN_PRO_MICRO" H 9450 4176 45  0000 C CNN
-F 2 "SPARKFUN_PRO_MICRO" H 9450 4150 20  0001 C CNN
+F 2 "OsseyPad:SPARKFUN_PRO_MICRO_OsseyPad" H 9450 4150 20  0001 C CNN
 F 3 "https://cdn.sparkfun.com/assets/f/d/8/0/d/ProMicro16MHzv2.pdf" H 9450 3350 50  0001 C CNN
 F 4 "XXX-00000" H 9450 4081 60  0000 C CNN "Field4"
