File: OsseyPad Rev 2.0/OsseyPad.kicad_pcb (KiCad board)
At the start: 2 copper layers, 157 x 148 mm, 83 parts, among them SW1 Rotary_Encoder_Switch

Commit message: Worked on with 2.0
Parts:
- added B1: SPARKFUN_PRO_MICRO, Boards:SPARKFUN_PRO_MICRO, B.Cu at (108.1, 90.4)
- C1, C2: value 100n -> 0.1 uf; footprint Capacitor_SMD:C_0603_1608Metric -> Capacitor_THT:C_Axial_L5.1mm_D3.1mm_P7.50mm_Horizontal; moved to B.Cu
- R1, R2, R3, R4: footprint Resistor_SMD:R_0603_1608Metric -> Resistor_THT:R_Axial_DIN0207_L6.3mm_D2.5mm_P7.62mm_Horizontal; moved to B.Cu
- moved C2 130.1 mm to (202.6, 78.8), turned to 270 degrees
- moved R3 128.9 mm to (206.0, 86.4), turned to 90 degrees
- moved R1 128.8 mm to (209.1, 78.8), turned to 270 degrees
- moved MX35 124.2 mm to (188.1, 152.4), turned to 270 degrees
- moved R4 117.7 mm to (206.4, 104.4), turned to 270 degrees
- moved MX36 114.3 mm to (188.1, 190.5), turned to 270 degrees
- moved R2 104.5 mm to (209.5, 112.0), turned to 90 degrees
- moved C1 100.8 mm to (203.1, 112.0), turned to 90 degrees
- moved D19 0.48 mm to (140.5, 152.4)
- moved D20 0.48 mm to (159.5, 152.4)
- moved D5 0.29 mm to (216.4, 85.7)
Connections:
- net +5V renamed +3V3
- net COL3+ renamed COL1+
- D10 pad 2: ROW3+ -> Net-(D10-Pad2)
- D16 pad 2: Net-(D16-Pad2) -> ROW4+
- D22 pad 2: ROW3ENTER -> Net-(D22-Pad2)
- D24 pad 2: Net-(D24-Pad2) -> ROW3ENTER
- MX15 pad 2: Net-(D16-Pad2) -> ROW4+
- MX21 pad 2: ROW3ENTER -> Net-(D22-Pad2)
- MX23 pad 2: Net-(D24-Pad2) -> ROW3ENTER
- MX35 pad 2: ROW3+ -> ROW4+
- MX9 pad 2: ROW3+ -> Net-(D10-Pad2)
Routing:
- net ROW5: track 0.00 -> 124.5 mm
- net COL1+: track 0.00 -> 121.9 mm
- net COL1: track 0.00 -> 121.8 mm
- net ROW3: track 0.00 -> 116.5 mm
- net ROW4: track 0.00 -> 114.3 mm
- net ROW2: track 0.00 -> 114.3 mm
- net ROW1: track 0.00 -> 114.3 mm
- net COL2: track 0.00 -> 109.5 mm
- net COL3: track 0.00 -> 104.8 mm
- net COL5: track 0.00 -> 104.2 mm
- net ROW0: track 0.00 -> 79.2 mm
- net COL0: track 0.00 -> 76.2 mm
- net ROW4+: track 0.00 -> 27.5 mm
- net ROW3ENTER: track 0.00 -> 27.5 mm
- net ROW50: track 0.00 -> 18.0 mm
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- added copper zone on F.Cu, net +3V3
- removed copper zone on F.Cu, net (none)
Other:
- net class Default: clearance 0.19 -> 0.2
- rule trace_clearance: 0.19 -> 0.2

Commit message: Worked on Rev 2.0.
Parts:
- moved C1 0.46 mm to (202.6, 111.9)
- moved R2 0.46 mm to (209.0, 112.0)
- moved R4 0.46 mm to (206.0, 104.4)
- moved B1 0.30 mm to (108.0, 90.2)
Connections:
- net ROW3ENTER renamed ROW4ENTER
- net ROW4+ renamed ROW2+
- B1 pad 10: Net-(B1-Pad10) -> COL2
- B1 pad 11: Net-(B1-Pad11) -> COL1
- B1 pad 12: Net-(B1-Pad12) -> ENC_1_B
- B1 pad 13: Net-(B1-Pad13) -> COL0
- B1 pad 16: Net-(B1-Pad16) -> ROW1
- B1 pad 17: Net-(B1-Pad17) -> ROW2
- B1 pad 18: Net-(B1-Pad18) -> ROW3
- B1 pad 19: Net-(B1-Pad19) -> ROW4
- B1 pad 20: Net-(B1-Pad20) -> ROW5
- B1 pad 21: Net-(B1-Pad21) -> +5V
- B1 pad 23: Net-(B1-Pad23) -> GND
- B1 pad 3: Net-(B1-Pad3) -> GND
- B1 pad 4: Net-(B1-Pad4) -> GND
- B1 pad 5: Net-(B1-Pad5) -> ENC_1_A
- B1 pad 6: Net-(B1-Pad6) -> ROW0
- B1 pad 7: Net-(B1-Pad7) -> COL5
- B1 pad 8: Net-(B1-Pad8) -> COL4
- B1 pad 9: Net-(B1-Pad9) -> COL3
- MX15 pad 1: COL1+ -> COL4
- MX21 pad 1: COL1+ -> COL4
- MX23 pad 1: COL1+ -> COL4
- MX33 pad 1: COL1+ -> COL4
- MX35 pad 1: COL1+ -> COL4
- MX36 pad 1: COL1+ -> COL4
- MX4 pad 1: COL1+ -> COL4
- MX9 pad 1: COL1+ -> COL4
- R1 pad 1: +3V3 -> +5V
- R2 pad 1: +3V3 -> +5V
Routing:
- net COL4: track 0.00 -> 208.1 mm
- net +5V: track 0.00 -> 174.4 mm
- net GND: track 4.79 -> 169.8 mm, vias 3 -> 4
- net ROW5: track 124.5 -> 257.3 mm
- net COL5: track 104.2 -> 231.3 mm
- net COL1+: track 121.9 -> 0.00 mm
- net ROW4: track 114.3 -> 225.0 mm
- net ENC_1_A: track 3.38 -> 94.0 mm
- net ENC_1_B: track 3.41 -> 93.1 mm
- net ROW3: track 116.5 -> 205.0 mm
- net COL3: track 104.8 -> 173.0 mm
- net ROW2: track 114.3 -> 180.6 mm
- net COL2: track 109.5 -> 158.9 mm
- net ROW1: track 114.3 -> 158.5 mm
- net ROW0: track 79.2 -> 105.9 mm
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- added copper zone on F.Cu, net (none)
- removed copper zone on F.Cu, net +3V3
Other:
- net class Default: trace_width 0.25 -> 0.3

Commit message: Worked on the pcb design.
Parts:
- B1: footprint Boards:SPARKFUN_PRO_MICRO -> OsseyPad:SPARKFUN_PRO_MICRO_OsseyPad
- moved D15 2.38 mm to (178.6, 133.3), turned to 180 degrees
- moved D28 2.38 mm to (178.6, 171.4), turned to 180 degrees
Routing:
- net GND: track 169.8 -> 167.7 mm, vias 4 -> 2
- net ROW4: track 225.0 -> 227.0 mm
- net ROW2: track 180.6 -> 182.6 mm
- net Net-(D28-Pad2): track 6.20 -> 4.51 mm
- net Net-(D15-Pad2): track 6.19 -> 4.71 mm
- net ENC_1_A: track 94.0 -> 95.1 mm
- net ROW0: track 105.9 -> 106.9 mm
- net ENC_1_B: track 93.1 -> 92.2 mm

Commit message: Updated the PCB for rev 2.0.
Parts:
- moved D10 4.48 mm to (200.0, 118.8)
- moved C2 1.22 mm to (201.4, 78.8)
- moved C1 1.19 mm to (201.4, 111.9)
- moved R3 0.60 mm to (205.4, 86.4)
- moved R4 0.58 mm to (205.4, 104.4)
Routing:
- net COL4: track 208.1 -> 214.1 mm
- net ROW1: track 158.5 -> 163.2 mm
- net Net-(D10-Pad2): track 10.7 -> 14.4 mm
- net ROW0: track 106.9 -> 105.9 mm
- net ENC_1_B: track 92.2 -> 91.6 mm
- net Net-(R1-Pad2): track 9.77 -> 10.4 mm
- net ENC_1_A: track 95.1 -> 94.5 mm
- net Net-(R2-Pad2): track 9.83 -> 10.4 mm

Commit message: Worked on rev 2.0.
Parts:
- removed B1: SPARKFUN_PRO_MICRO, OsseyPad:SPARKFUN_PRO_MICRO_OsseyPad
- added U1: Elite-C, Keebio-Parts:Elite-C-castellated-29pin-holes, B.Cu at (106.0, 91.5)
- moved D15 14.8 mm to (163.8, 133.3), turned to 0 degrees
- moved D28 14.8 mm to (163.8, 171.4), turned to 0 degrees
Routing:
- net GND: track 167.7 -> 109.0 mm
- net +5V: track 174.4 -> 148.6 mm
- net COL4: track 214.1 -> 192.2 mm
- net COL5: track 231.3 -> 211.6 mm
- net ENC_1_A: track 94.5 -> 77.6 mm
- net COL0: track 92.9 -> 82.1 mm
- net ROW0: track 105.9 -> 95.6 mm
- net COL1: track 140.4 -> 130.4 mm
- net COL2: track 158.9 -> 150.6 mm
- net ROW1: track 163.2 -> 155.7 mm
- net ROW5: track 257.3 -> 264.8 mm
- net COL3: track 173.0 -> 166.3 mm
- net ROW4: track 227.0 -> 230.6 mm
- net ENC_1_B: track 91.6 -> 88.3 mm
- net ROW2: track 182.6 -> 180.8 mm
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Other:
- net class Default removed

Commit message: Worked on pcb and case for 2.0.
Parts:
- MX1, MX10, MX11, MX12, MX13, MX14, MX15, MX16, MX17, MX18, MX19, MX2, MX20, MX21, MX22, MX23, MX24, MX25, MX26, MX27, MX28, MX29, MX3, MX30, MX31, MX32, MX33, MX34, MX4, MX5, MX6, MX7, MX8, MX9: footprint MX_Only:MXOnly-1U-NoLED -> MX_Only:MXOnly-1U-NoLED_Edit1
- SW1: footprint Rotary_Encoder:RotaryEncoder_Alps_EC11E-Switch_Vertical_H20mm_CircularMountingHoles -> OsseyPad:RotaryEncoder_Alps_EC11E-Switch_Vertical_H20mm_CircularMountingHoles_Edit1
- U1: footprint Keebio-Parts:Elite-C-castellated-29pin-holes -> OsseyPad:Elite-C-castellated-29pin-holes_Edit1
- moved D31 20.2 mm to (140.5, 188.1)
- moved SW1 7.53 mm to (216.7, 95.2)
- moved H4 1.70 mm to (232.0, 215.6)
- moved H2 1.70 mm to (232.0, 79.6)
- moved H3 1.70 mm to (87.0, 215.6)
- moved H1 1.70 mm to (87.0, 79.6)
- moved D5 0.33 mm to (216.1, 85.7)
- moved U1 0.29 mm to (105.9, 91.7), turned to 180 degrees
- moved C2 0.21 mm to (201.5, 78.6)
- moved R1 0.21 mm to (209.2, 78.6)
- moved R3 0.21 mm to (205.5, 86.2)
- moved D15 0.15 mm to (164.0, 133.3)
- moved D28 0.15 mm to (164.0, 171.4)
- moved C1 0.14 mm to (201.5, 111.8)
- moved R2 0.14 mm to (209.2, 111.9)
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Routing:
- net GND: track 109.0 -> 195.9 mm, vias 2 -> 6
- net ENC_1_A: track 77.6 -> 20.3 mm
- net COL5: track 211.6 -> 243.1 mm
- net COL4: track 192.2 -> 218.9 mm
- net COL1: track 130.4 -> 147.5 mm
- net +5V: track 148.6 -> 164.8 mm
- net COL2: track 150.6 -> 163.4 mm
- net ROW0: track 95.6 -> 106.4 mm
- net COL0: track 82.1 -> 92.1 mm
- net COL3: track 166.3 -> 175.1 mm
- net ROW50: track 18.0 -> 12.0 mm
- net ROW5: track 264.8 -> 259.0 mm
- net ENC_1_B: track 88.3 -> 93.4 mm
- net ROW1: track 155.7 -> 157.5 mm
- net ROW2: track 180.8 -> 180.1 mm
- added copper zone on F.Cu, net GND
- removed copper zone on F.Cu, net (none)

Commit message: Worked on pcb and case.
Parts:
- C1, C2: footprint Capacitor_THT:C_Axial_L5.1mm_D3.1mm_P7.50mm_Horizontal -> Capacitor_THT:C_Disc_D3.0mm_W2.0mm_P2.50mm
Routing:
- net ENC_1_A: track 20.3 -> 100.1 mm
- net GND: track 195.9 -> 213.9 mm
- net +5V: track 164.8 -> 177.3 mm
- net ROW0: track 106.4 -> 104.2 mm
- net COL5: track 243.1 -> 242.0 mm

Commit message: Worked on Rev 2.0.
Parts:
- added G***: LOGO, OsseyPad:HelloToHorse, B.Cu at (202.5, 212.7)
Other:
- board text added: "Designed by Osku Väyrynen 10/2/2021 Rev 2.0"
- board text added: "JLCJLCJLCJLC"
- board text added: "OsseyPad Rev. 2.0"
