File: OsseyPad Rev 2.0/OsseyPad.kicad_sch (KiCad schematic)
At the start: 84 parts, among them SW1 Rotary_Encoder_Switch, U1 Elite-C

Commit message: Worked on pcb and case for 2.0.
Parts:
- MX1, MX10, MX11, MX12, MX13, MX14, MX15, MX16, MX17, MX18, MX19, MX2, MX20, MX21, MX22, MX23, MX24, MX25, MX26, MX27, MX28, MX29, MX3, MX30, MX31, MX32, MX33, MX34, MX4, MX5, MX6, MX7, MX8, MX9: footprint MX_Only:MXOnly-1U-NoLED -> MX_Only:MXOnly-1U-NoLED_Edit1
- SW1: footprint Rotary_Encoder:RotaryEncoder_Alps_EC11E-Switch_Vertical_H20mm_CircularMountingHoles -> OsseyPad:RotaryEncoder_Alps_EC11E-Switch_Vertical_H20mm_CircularMountingHoles_Edit1
- U1: footprint Keebio-Parts:Elite-C-castellated-29pin-holes -> OsseyPad:Elite-C-castellated-29pin-holes_Edit1
Connections:
- no-connect marks 0 -> 11

Commit message: Worked on pcb and case.
Parts:
- C1, C2: footprint Capacitor_THT:C_Axial_L5.1mm_D3.1mm_P7.50mm_Horizontal -> Capacitor_THT:C_Disc_D3.0mm_W2.0mm_P2.50mm
Changed lines of the file:
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@@
       (effects (font (size 1.27 1.27)) (justify left))
     )
-    (property "Footprint" "Capacitor_THT:C_Axial_L5.1mm_D3.1mm_P7.50mm_Horizontal" (id 2) (at 62.23 48.26 0)
+    (property "Footprint" "Capacitor_THT:C_Disc_D3.0mm_W2.0mm_P2.50mm" (id 2) (at 62.23 48.26 0)
       (effects (font (size 1.27 1.27)) hide)
     )
@@
       (effects (font (size 1.27 1.27)) (justify left))
     )
-    (property "Footprint" "Capacitor_THT:C_Axial_L5.1mm_D3.1mm_P7.50mm_Horizontal" (id 2) (at 72.39 48.26 0)
+    (property "Footprint" "Capacitor_THT:C_Disc_D3.0mm_W2.0mm_P2.50mm" (id 2) (at 72.39 48.26 0)
       (effects (font (size 1.27 1.27)) hide)
     )
@@
     )
     (path "/00000000-0000-0000-0000-00006006944a"
-      (reference "C1") (unit 1) (value "0.1 uf") (footprint "Capacitor_THT:C_Axial_L5.1mm_D3.1mm_P7.50mm_Horizontal")
+      (reference "C1") (unit 1) (value "0.1 uf") (footprint "Capacitor_THT:C_Disc_D3.0mm_W2.0mm_P2.50mm")
     )
     (path "/00000000-0000-0000-0000-0000600670a6"
-      (reference "C2") (unit 1) (value "0.1 uf") (footprint "Capacitor_THT:C_Axial_L5.1mm_D3.1mm_P7.50mm_Horizontal")
+      (reference "C2") (unit 1) (value "0.1 uf") (footprint "Capacitor_THT:C_Disc_D3.0mm_W2.0mm_P2.50mm")
     )
     (path "/00000000-0000-0000-0000-00005ff933be"

Commit message: Updated the pcb and case.
Parts:
- R1, R2, R3, R4: footprint Resistor_THT:R_Axial_DIN0207_L6.3mm_D2.5mm_P7.62mm_Horizontal -> Resistor_THT:R_Axial_DIN0309_L9.0mm_D3.2mm_P12.70mm_Horizontal
Changed lines of the file:
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@@
-    (stroke (width 0) (type solid) (color 0 0 0 0))
-  )
-  (wire (pts (xy 66.04 87.63) (xy 80.01 87.63))
     (stroke (width 0) (type solid) (color 0 0 0 0))
   )
@@
   )
   (wire (pts (xy 80.01 83.82) (xy 80.01 87.63))
+    (stroke (width 0) (type solid) (color 0 0 0 0))
+  )
+  (wire (pts (xy 80.01 87.63) (xy 66.04 87.63))
     (stroke (width 0) (type solid) (color 0 0 0 0))
   )
@@
     (property "Reference" "R3" (id 0) (at 78.74 38.1 90))
     (property "Value" "10K" (id 1) (at 78.74 35.433 90))
-    (property "Footprint" "Resistor_THT:R_Axial_DIN0207_L6.3mm_D2.5mm_P7.62mm_Horizontal" (id 2) (at 78.74 38.1 0)
+    (property "Footprint" "Resistor_THT:R_Axial_DIN0309_L9.0mm_D3.2mm_P12.70mm_Horizontal" (id 2) (at 78.74 38.1 0)
       (effects (font (size 1.27 1.27)) hide)
     )
@@
     (property "Reference" "R4" (id 0) (at 78.74 43.18 90))
     (property "Value" "10K" (id 1) (at 78.74 40.64 90))
-    (property "Footprint" "Resistor_THT:R_Axial_DIN0207_L6.3mm_D2.5mm_P7.62mm_Horizontal" (id 2) (at 78.74 43.18 0)
+    (property "Footprint" "Resistor_THT:R_Axial_DIN0309_L9.0mm_D3.2mm_P12.70mm_Horizontal" (id 2) (at 78.74 43.18 0)
       (effects (font (size 1.27 1.27)) hide)
     )
@@
       (effects (font (size 1.27 1.27)) (justify left))
     )
-    (property "Footprint" "Resistor_THT:R_Axial_DIN0207_L6.3mm_D2.5mm_P7.62mm_Horizontal" (id 2) (at 85.09 34.29 0)
+    (property "Footprint" "Resistor_THT:R_Axial_DIN0309_L9.0mm_D3.2mm_P12.70mm_Horizontal" (id 2) (at 85.09 34.29 0)
       (effects (font (size 1.27 1.27)) hide)
     )
@@
       (effects (font (size 1.27 1.27)) (justify left))
     )
-    (property "Footprint" "Resistor_THT:R_Axial_DIN0207_L6.3mm_D2.5mm_P7.62mm_Horizontal" (id 2) (at 91.44 34.29 0)
+    (property "Footprint" "Resistor_THT:R_Axial_DIN0309_L9.0mm_D3.2mm_P12.70mm_Horizontal" (id 2) (at 91.44 34.29 0)
       (effects (font (size 1.27 1.27)) hide)
     )
@@
     )
     (path "/00000000-0000-0000-0000-00005ffbd2ee"
-      (reference "R1") (unit 1) (value "10K") (footprint "Resistor_THT:R_Axial_DIN0207_L6.3mm_D2.5mm_P7.62mm_Horizontal")
+      (reference "R1") (unit 1) (value "10K") (footprint "Resistor_THT:R_Axial_DIN0309_L9.0mm_D3.2mm_P12.70mm_Horizontal")
     )
     (path "/00000000-0000-0000-0000-00005ffd944d"
-      (reference "R2") (unit 1) (value "10K") (footprint "Resistor_THT:R_Axial_DIN0207_L6.3mm_D2.5mm_P7.62mm_Horizontal")
+      (reference "R2") (unit 1) (value "10K") (footprint "Resistor_THT:R_Axial_DIN0309_L9.0mm_D3.2mm_P12.70mm_Horizontal")
     )
     (path "/00000000-0000-0000-0000-000060002259"
-      (reference "R3") (unit 1) (value "10K") (footprint "Resistor_THT:R_Axial_DIN0207_L6.3mm_D2.5mm_P7.62mm_Horizontal")
+      (reference "R3") (unit 1) (value "10K") (footprint "Resistor_THT:R_Axial_DIN0309_L9.0mm_D3.2mm_P12.70mm_Horizontal")
     )
     (path "/00000000-0000-0000-0000-000060049e0c"
-      (reference "R4") (unit 1) (value "10K") (footprint "Resistor_THT:R_Axial_DIN0207_L6.3mm_D2.5mm_P7.62mm_Horizontal")
+      (reference "R4") (unit 1) (value "10K") (footprint "Resistor_THT:R_Axial_DIN0309_L9.0mm_D3.2mm_P12.70mm_Horizontal")
     )
     (path "/00000000-0000-0000-0000-00005feeb78a"
